File: pcb/keypad.kicad_pcb (KiCad board)
At the start: 2 copper layers, 148 x 103 mm, 55 parts, among them J1 Conn_02x06_Odd_Even, SW1 SW_Push, SW10 SW_Push, SW11 SW_Push, SW12 SW_Push, SW13 SW_Push, SW14 SW_Push, SW15 SW_Push, SW16 SW_Push, SW17 SW_Push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

Commit message: - Marked NC pins  - Updated diode symbols
Parts:
- U1: value ProMicro -> kb2040
Changed lines of the file:
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@@
       (net 3 "/Col1") (pinfunction "Pin_6") (pintype "passive"))
     (pad "7" thru_hole oval (at 0 7.62 180) (size 1.7 1.7) (drill 1) (layers *.Cu *.Mask)
-      (net 42 "unconnected-(J1-Pad7)") (pinfunction "Pin_7") (pintype "passive"))
+      (net 42 "unconnected-(J1-Pad7)") (pinfunction "Pin_7") (pintype "passive+no_connect"))
     (pad "8" thru_hole oval (at 2.54 7.62 180) (size 1.7 1.7) (drill 1) (layers *.Cu *.Mask)
       (net 5 "/Col2") (pinfunction "Pin_8") (pintype "passive"))
     (pad "9" thru_hole oval (at 0 10.16 180) (size 1.7 1.7) (drill 1) (layers *.Cu *.Mask)
-      (net 43 "unconnected-(J1-Pad9)") (pinfunction "Pin_9") (pintype "passive"))
+      (net 43 "unconnected-(J1-Pad9)") (pinfunction "Pin_9") (pintype "passive+no_connect"))
     (pad "10" thru_hole oval (at 2.54 10.16 180) (size 1.7 1.7) (drill 1) (layers *.Cu *.Mask)
       (net 7 "/Col3") (pinfunction "Pin_10") (pintype "passive"))
@@
       (effects (font (size 1.27 1.524) (thickness 0.2032)))
     )
-    (fp_text value "ProMicro" (at 0 0 -90) (layer "F.SilkS") hide
+    (fp_text value "kb2040" (at 0 0 -90) (layer "F.SilkS") hide
       (effects (font (size 1.27 1.524) (thickness 0.2032)))
     )
@@
     (fp_line (start -3.81 -19.304) (end 3.556 -19.304) (layer "Dwgs.User") (width 0.2))
     (pad "1" thru_hole rect (at -7.62 -13.97 180) (size 1.7526 1.7526) (drill 1.0922) (layers *.Cu *.SilkS *.Mask)
-      (net 23 "unconnected-(U1-Pad1)") (pinfunction "D+") (pintype "bidirectional"))
+      (net 23 "unconnected-(U1-Pad1)") (pinfunction "D+") (pintype "bidirectional+no_connect"))
     (pad "2" thru_hole circle (at -7.62 -11.43 180) (size 1.7526 1.7526) (drill 1.0922) (layers *.Cu *.SilkS *.Mask)
-      (net 20 "unconnected-(U1-Pad2)") (pinfunction "D0") (pintype "bidirectional"))
+      (net 20 "unconnected-(U1-Pad2)") (pinfunction "D0") (pintype "bidirectional+no_connect"))
     (pad "3" thru_hole circle (at -7.62 -8.89 180) (size 1.7526 1.7526) (drill 1.0922) (layers *.Cu *.SilkS *.Mask)
-      (net 47 "unconnected-(U1-Pad3)") (pinfunction "D1") (pintype "bidirectional"))
+      (net 47 "unconnected-(U1-Pad3)") (pinfunction "D1") (pintype "bidirectional+no_connect"))
     (pad "4" thru_hole circle (at -7.62 -6.35 180) (size 1.7526 1.7526) (drill 1.0922) (layers *.Cu *.SilkS *.Mask)
       (net 21 "/GND") (pinfunction "GND") (pintype "bidirectional"))
@@
       (net 21 "/GND") (pinfunction "GND") (pintype "bidirectional"))
     (pad "6" thru_hole circle (at -7.62 -1.27 180) (size 1.7526 1.7526) (drill 1.0922) (layers *.Cu *.SilkS *.Mask)
-      (net 39 "unconnected-(U1-Pad6)") (pinfunction "D2") (pintype "bidirectional"))
+      (net 39 "unconnected-(U1-Pad6)") (pinfunction "D2") (pintype "bidirectional+no_connect"))
     (pad "7" thru_hole circle (at -7.62 1.27 180) (size 1.7526 1.7526) (drill 1.0922) (layers *.Cu *.SilkS *.Mask)
-      (net 48 "unconnected-(U1-Pad7)") (pinfunction "D3") (pintype "bidirectional"))
+      (net 48 "unconnected-(U1-Pad7)") (pinfunction "D3") (pintype "bidirectional+no_connect"))
     (pad "8" thru_hole circle (at -7.62 3.81 180) (size 1.7526 1.7526) (drill 1.0922) (layers *.Cu *.SilkS *.Mask)
       (net 41 "/Row5") (pinfunction "D4") (pintype "bidirectional"))
@@
       (net 15 "/Row0") (pinfunction "D9") (pintype "bidirectional"))
     (pad "14" thru_hole circle (at 7.62 -13.97 180) (size 1.7526 1.7526) (drill 1.0922) (layers *.Cu *.SilkS *.Mask)
-      (net 49 "unconnected-(U1-Pad14)") (pinfunction "D-") (pintype "bidirectional"))
+      (net 49 "unconnected-(U1-Pad14)") (pinfunction "D-") (pintype "bidirectional+no_connect"))
     (pad "15" thru_hole circle (at 7.62 -11.43 180) (size 1.7526 1.7526) (drill 1.0922) (layers *.Cu *.SilkS *.Mask)
-      (net 50 "unconnected-(U1-Pad15)") (pinfunction "RAW") (pintype "bidirectional"))
+      (net 50 "unconnected-(U1-Pad15)") (pinfunction "RAW") (pintype "bidirectional+no_connect"))
     (pad "16" thru_hole circle (at 7.62 -8.89 180) (size 1.7526 1.7526) (drill 1.0922) (layers *.Cu *.SilkS *.Mask)
       (net 21 "/GND") (pinfunction "GND") (pintype "bidirectional"))
@@
       (net 46 "/3.3v") (pinfunction "3.3v") (pintype "bidirectional"))
     (pad "19" thru_hole circle (at 7.62 -1.27 180) (size 1.7526 1.7526) (drill 1.0922) (layers *.Cu *.SilkS *.Mask)
-      (net 44 "unconnected-(U1-Pad19)") (pinfunction "A3/29") (pintype "bidirectional"))
+      (net 44 "unconnected-(U1-Pad19)") (pinfunction "A3/29") (pintype "bidirectional+no_connect"))
     (pad "20" thru_hole circle (at 7.62 1.27 180) (size 1.7526 1.7526) (drill 1.0922) (layers *.Cu *.SilkS *.Mask)
-      (net 45 "unconnected-(U1-Pad20)") (pinfunction "A2/28") (pintype "bidirectional"))
+      (net 45 "unconnected-(U1-Pad20)") (pinfunction "A2/28") (pintype "bidirectional+no_connect"))
     (pad "21" thru_hole circle (at 7.62 3.81 180) (size 1.7526 1.7526) (drill 1.0922) (layers *.Cu *.SilkS *.Mask)
       (net 1 "/Col0") (pinfunction "A1/27") (pintype "bidirectional"))
