File: thumb_pod/thumb_pod.kicad_pcb (KiCad board)
At the start: 2 copper layers, 93 x 56 mm, 55 parts, among them J1 Conn_02x06_Odd_Even, J2 Conn_02x06_Odd_Even, J3 Conn_02x06_Odd_Even, SW1 SW_Push, SW10 SW_Push, SW2 SW_Push, SW3 SW_Push, SW4 SW_Push, SW5 SW_Push, SW6 SW_Push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

Commit message: - Removed "micro" thumb pod  - Added kailh gm microswitch footprint  - Switch to kail gm microswitches for the "mini" thumb pod  - Reduced size of joystick silkscreen
Parts:
- removed D10, D11, D12, D9: 1N4148, Diode_THT:D_DO-35_SOD27_P7.62mm_Horizontal
- removed H4, H5: MountingHole, MountingHole:MountingHole_3.2mm_M3
- removed J2: Conn_02x06_Odd_Even, keypad:PinHeader_2x06_P2.54mm_Horizontal
- removed U2: RKJXM1015004, thumb_pod:RKJXM1015004
- removed the mouse-bite-2mm-slot at (61.8, 54.0)
- removed the mouse-bite-2mm-slot at (85.0, 57.0)
- removed the mouse-bite-2mm-slot at (85.0, 64.0)
- removed the mouse-bite-2mm-slot at (82.0, 54.0)
- removed the mouse-bite-2mm-slot at (85.0, 78.0)
- removed the mouse-bite-2mm-slot at (85.0, 71.0)
- removed the mouse-bite-2mm-slot at (55.0, 54.0)
- removed the mouse-bite-2mm-slot at (68.5, 54.0)
- removed the mouse-bite-2mm-slot at (75.2, 54.0)
- SW10, SW9: footprint Button_Switch_THT:SW_PUSH_6mm -> keypad:kailh_gm_microswitch
- moved D16 29.1 mm to (54.6, 37.1), turned to -90 degrees
- moved H6 23.2 mm to (80.4, 49.5)
- moved SW10 21.3 mm to (70.0, 52.0), turned to 90 degrees
- moved H7 18.4 mm to (62.1, 27.7)
- moved D17 14.9 mm to (63.2, 37.2), turned to -90 degrees
- moved D13 12.2 mm to (70.8, 47.7), turned to 180 degrees
- moved D18 8.90 mm to (54.5, 52.4)
- moved D15 8.82 mm to (64.0, 33.8), turned to 180 degrees
- moved SW9 6.56 mm to (59.0, 41.7)
- moved J3 5.45 mm to (69.5, 30.9)
- moved U3 1.66 mm to (72.3, 40.0)
- moved D14 0.58 mm to (82.2, 33.8)
Routing:
- net Net-(J2-Pad4): track 29.6 -> 0.00 mm
- net Net-(J2-Pad10): track 25.3 -> 0.00 mm
- net Net-(J2-Pad6): track 17.9 -> 0.00 mm
- net Net-(J2-Pad8): track 16.5 -> 0.00 mm
- net unconnected-(U2-Pad3): track 16.1 -> 0.00 mm
- net Net-(U2-Pad2): track 15.0 -> 0.00 mm
- net Net-(D9-Pad2): track 14.0 -> 0.00 mm
- net Net-(D17-Pad2): track 17.0 -> 5.83 mm
- net Net-(J2-Pad3): track 9.60 -> 0.00 mm
- net Net-(D13-Pad1): track 37.2 -> 45.9 mm
- net Net-(D17-Pad1): track 30.9 -> 23.4 mm
- net Net-(U2-Pad5): track 6.89 -> 0.00 mm
- net Net-(D13-Pad2): track 8.67 -> 14.4 mm
- net Net-(D14-Pad1): track 50.0 -> 55.7 mm
- net Net-(U2-Pad7): track 4.87 -> 0.00 mm
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- removed copper zone on B.Cu, net /GND_u
- removed copper zone on F.Cu, net /GND_u
Other:
- outline, holes or cut-outs redrawn
- board text removed: "kp13 Thumb Pod Micro v0.1"

Commit message: - Updated the kailh gm switch footprint to match the SPDT symbol  - Updated the mini thumb pod switches to allow them to be placed in either orientation
Parts:
- SW10, SW9: value SW_Push -> SW_Push_SPDT
- moved SW10 0.18 mm to (69.9, 51.9)
- moved SW9 0.11 mm to (59.0, 41.8)
Connections:
- SW10 pad 2: Net-(D18-Pad2) -> Net-(J3-Pad5)
- SW10 pad 3: (no net) -> Net-(D18-Pad2)
- SW9 pad 2: Net-(D16-Pad2) -> Net-(J3-Pad5)
- SW9 pad 3: (no net) -> Net-(D16-Pad2)
Routing:
- net Net-(J3-Pad5): track 35.7 -> 51.7 mm
- net /GND_m: vias 10 -> 15
